Commit message: Did some minor fixes, code should work!

File: flex_gazebo/urdf/iiwa7.urdf.xacro (robot description, xacro)
@@ -11,7 +11,7 @@
   <xacro:arg name="origin_xyz" default="0 0 0"/>
   <xacro:arg name="origin_rpy" default="0 0 0"/>
-  <xacro:arg name="rs_origin_xyz" default="0 0.6 1.2"/>
-  <xacro:arg name="rs_origin_rpy" default="3.1415 1.57 -1.57"/>
   <xacro:arg name="camera_name" default="camera"/>
+  <xacro:arg name="camera_origin_xyz" default="0 0.6 1.2"/>
+  <xacro:arg name="camera_origin_rpy" default="3.1415 1.57 -1.57"/>
   <xacro:arg name="use_nominal_extrinsics" default="true"/>
   <!-- Fix to world just for testing -->
@@ -21,6 +21,6 @@
     <origin xyz="$(arg origin_xyz)" rpy="$(arg origin_rpy)" />
   </xacro:iiwa7>
-  <xacro:sensor_d435 parent="world" name="$(arg camera_name)" use_nominal_extrinsics="$(arg use_nominal_extrinsics)"> <!-- use_nominal_extrinsics="$(arg use_nominal_extrinsics)" -->
-    <origin xyz="$(arg rs_origin_xyz)" rpy="$(arg rs_origin_rpy)" />
+  <xacro:sensor_d435 parent="world" name="$(arg camera_name)" use_nominal_extrinsics="$(arg use_nominal_extrinsics)">
+    <origin xyz="$(arg camera_origin_xyz)" rpy="$(arg camera_origin_rpy)" />
   </xacro:sensor_d435>
 </robot>

Commit message: tomato is now loaded via urdf, we can pass parameters to these file, in the future this can be used to spawn tomatoes at a random loaction.

File: flex_gazebo/urdf/iiwa7.urdf.xacro (robot description, xacro)
@@ -5,14 +5,12 @@
   <!--Import the lbr iiwa macro -->
   <xacro:include filename="$(find iiwa_description)/urdf/iiwa7.xacro"/>
-  <!-- import the camera -->
-  <xacro:include filename="$(find realsense2_description)/urdf/_d435.urdf.xacro" />
+  <!-- import the tomato -->
+  <xacro:include filename="$(find flex_gazebo)/urdf/tomato.xacro" />
   <xacro:arg name="hardware_interface" default="PositionJointInterface"/>
   <xacro:arg name="robot_name" default="iiwa"/>
   <xacro:arg name="origin_xyz" default="0 0 0"/>
   <xacro:arg name="origin_rpy" default="0 0 0"/>
-  <xacro:arg name="camera_name" default="camera"/>
-  <xacro:arg name="camera_origin_xyz" default="0 0.6 1.2"/>
-  <xacro:arg name="camera_origin_rpy" default="3.1415 1.57 -1.57"/>
-  <xacro:arg name="use_nominal_extrinsics" default="true"/>
+  <xacro:arg name="tomato_origin_xyz" default="-0.2 0.4 0.26"/>
+  <xacro:arg name="tomato_origin_rpy" default="0 0 0.3"/>
   <!-- Fix to world just for testing -->
   <link name="world"/>
@@ -21,7 +19,7 @@
     <origin xyz="$(arg origin_xyz)" rpy="$(arg origin_rpy)" />
   </xacro:iiwa7>
-  <xacro:sensor_d435 parent="world" name="$(arg camera_name)" use_nominal_extrinsics="$(arg use_nominal_extrinsics)">
-    <origin xyz="$(arg camera_origin_xyz)" rpy="$(arg camera_origin_rpy)" />
-  </xacro:sensor_d435>
+  <xacro:tomato_2d>
+    <origin xyz="$(arg tomato_origin_xyz)" rpy="$(arg tomato_origin_rpy)" />
+  </xacro:tomato_2d>
 </robot>
 <!-- This does not belong here! -->

Commit message: Fixed some issues, now the robot moves again, however it goes to the wrong position. Likely some wrong transfomration applied to the camera

File: flex_gazebo/urdf/iiwa7.urdf.xacro (robot description, xacro)
@@ -5,10 +5,19 @@
   <!--Import the lbr iiwa macro -->
   <xacro:include filename="$(find iiwa_description)/urdf/iiwa7.xacro"/>
+  <!-- import the camera -->
+  <xacro:include filename="$(find realsense2_description)/urdf/_d435.urdf.xacro" />
   <!-- import the tomato -->
   <xacro:include filename="$(find flex_gazebo)/urdf/tomato.xacro" />
+  <!-- iiwa params-->
   <xacro:arg name="hardware_interface" default="PositionJointInterface"/>
   <xacro:arg name="robot_name" default="iiwa"/>
   <xacro:arg name="origin_xyz" default="0 0 0"/>
   <xacro:arg name="origin_rpy" default="0 0 0"/>
+  <!-- camera params-->
+  <xacro:arg name="camera_name" default="camera"/>
+  <xacro:arg name="camera_origin_xyz" default="0 0.6 1.2"/>
+  <xacro:arg name="camera_origin_rpy" default="3.1415 1.57 -1.57"/>
+  <xacro:arg name="use_nominal_extrinsics" default="true"/>
+  <!-- tomato params-->
   <xacro:arg name="tomato_origin_xyz" default="-0.2 0.4 0.26"/>
   <xacro:arg name="tomato_origin_rpy" default="0 0 0.3"/>
@@ -19,4 +28,9 @@
     <origin xyz="$(arg origin_xyz)" rpy="$(arg origin_rpy)" />
   </xacro:iiwa7>
+  <!-- camera -->
+  <xacro:sensor_d435 parent="world" name="$(arg camera_name)" use_nominal_extrinsics="$(arg use_nominal_extrinsics)">
+    <origin xyz="$(arg camera_origin_xyz)" rpy="$(arg camera_origin_rpy)" />
+  </xacro:sensor_d435>
+  <!-- tomato -->
   <xacro:tomato_2d>
     <origin xyz="$(arg tomato_origin_xyz)" rpy="$(arg tomato_origin_rpy)" />
