Commit message: add possibility to switch between end-effectors

File: flex_gazebo/urdf/gripper.urdf.xacro (robot description, xacro)
@@ -37,5 +37,5 @@
         <origin rpy="0.0 0 0" xyz="0 0 0"/>
         <geometry>
-            <mesh filename="package://urdf_tutorial/meshes/l_finger.dae"/>
+            <mesh filename="package://flex_gazebo/models/gripper/l_finger.dae"/>
         </geometry>
         </visual>
@@ -43,5 +43,5 @@
         <origin rpy="0.0 0 0" xyz="0 0 0"/>
         <geometry>
-            <mesh filename="package://urdf_tutorial/meshes/l_finger.dae"/>
+            <mesh filename="package://flex_gazebo/models/gripper/l_finger.dae"/>
         </geometry>
         </collision>
@@ -55,5 +55,5 @@
         <origin rpy="0.0 0 0" xyz="0.09137 0.00495 0"/>
         <geometry>
-            <mesh filename="package://urdf_tutorial/meshes/l_finger_tip.dae"/>
+            <mesh filename="package://flex_gazebo/models/gripper/l_finger_tip.dae"/>
         </geometry>
         </visual>
@@ -68,5 +68,5 @@
         <origin rpy="-3.1415 0 0" xyz="0 0 0"/>
         <geometry>
-            <mesh filename="package://urdf_tutorial/meshes/l_finger.dae"/>
+            <mesh filename="package://flex_gazebo/models/gripper/l_finger.dae"/>
         </geometry>
         </visual>
@@ -74,5 +74,5 @@
         <origin rpy="-3.1415 0 0" xyz="0 0 0"/>
         <geometry>
-            <mesh filename="package://urdf_tutorial/meshes/l_finger.dae"/>
+            <mesh filename="package://flex_gazebo/models/gripper/l_finger.dae"/>
         </geometry>
         </collision>
@@ -86,5 +86,5 @@
         <origin rpy="-3.1415 0 0" xyz="0.09137 0.00495 0"/>
         <geometry>
-            <mesh filename="package://urdf_tutorial/meshes/l_finger_tip.dae"/>
+            <mesh filename="package://flex_gazebo/models/gripper/l_finger_tip.dae"/>
         </geometry>
         </visual>
@@ -92,5 +92,5 @@
         <origin rpy="-3.1415 0 0" xyz="0.09137 0.00495 0"/>
         <geometry>
-            <mesh filename="package://urdf_tutorial/meshes/l_finger_tip.dae"/>
+            <mesh filename="package://flex_gazebo/models/gripper/l_finger_tip.dae"/>
         </geometry>
         </collision>

File: flex_gazebo/urdf/robot_gripper.urdf.xacro (robot description, xacro)
@@ -7,4 +7,6 @@
   <!-- import the camera -->
   <xacro:include filename="$(find realsense2_description)/urdf/_d435.urdf.xacro" />
+  <!-- import the end-effector -->
+  <xacro:include filename="$(find flex_gazebo)/urdf/gripper.urdf.xacro" />
   <!-- iiwa params-->
   <xacro:arg name="hardware_interface" default="PositionJointInterface"/>
@@ -27,4 +29,7 @@
     <origin xyz="$(arg camera_origin_xyz)" rpy="$(arg camera_origin_rpy)" />
   </xacro:sensor_d435>
+  <!-- end-effector -->
+  <xacro:endeffector>
+  </xacro:endeffector>
 </robot>
 <!-- This does not belong here! -->

Commit message: Added arg ee for choosing end effector

File: flex_gazebo/urdf/gripper.urdf.xacro (robot description, xacro)
@@ -1,107 +1,325 @@
 <?xml version="1.0"?>
-<!-- Here we define the robot, we named it "iiwa7_tool" -->
-<robot xmlns:xacro="http://www.ros.org/wiki/xacro" name="iiwa7">
-  <xacro:macro name="endeffector">
-    <!-- End-effector params -->
-    <property name="tool_mass" value="0.200" />
-    <property name="tool_joint_offset" value="0.00 0.00 0.00" />
-    <property name="tool_link_offset" value="0.2 0.00 0" />
-    <!--  Here we define a dummy joint between the tip of the iiwa7 and the base of the tool.
-    There is no offset between the two, that means the tool is attached at the robot flange. -->
-    <joint name="tool_joint" type="fixed">
-        <parent link="iiwa_link_ee" />
-        <child link = "gripper_pole" />
-        <origin xyz="${tool_joint_offset}" rpy="0 -${PI/2.0} 0" />
-    </joint>
-    <link name="gripper_pole">
-        <visual>
-        <geometry>
-            <cylinder length="0.05" radius="0.01"/>
-        </geometry>
-        <origin rpy="0 ${PI/2.0} 0 " xyz="0.025 0 0"/>
-        </visual>
-        <collision>
-        <geometry>
-            <cylinder length="0.05" radius="0.01"/>
-        </geometry>
-        <origin rpy="0 ${PI/2.0} 0 " xyz="0.025 0 0"/>
-        </collision>
-    </link>
-    <joint name="left_gripper_joint" type="fixed">
-        <origin rpy="0 0 0" xyz="0.05 0.01 0"/>
-        <parent link="gripper_pole"/>
-        <child link="left_gripper"/>
-    </joint>
-    <link name="left_gripper">
-        <visual>
-        <origin rpy="0.0 0 0" xyz="0 0 0"/>
-        <geometry>
-            <mesh filename="package://flex_gazebo/models/gripper/l_finger.dae"/>
-        </geometry>
-        </visual>
-        <collision>
-        <origin rpy="0.0 0 0" xyz="0 0 0"/>
-        <geometry>
-            <mesh filename="package://flex_gazebo/models/gripper/l_finger.dae"/>
-        </geometry>
-        </collision>
-    </link>
-    <joint name="left_tip_joint" type="fixed">
-        <parent link="left_gripper"/>
-        <child link="left_tip"/>
-    </joint>
-    <link name="left_tip">
-        <visual>
-        <origin rpy="0.0 0 0" xyz="0.09137 0.00495 0"/>
-        <geometry>
-            <mesh filename="package://flex_gazebo/models/gripper/l_finger_tip.dae"/>
-        </geometry>
-        </visual>
-    </link>
-    <joint name="right_gripper_joint" type="fixed">
-        <origin rpy="0 0 0" xyz="0.05 -0.01 0"/>
-        <parent link="gripper_pole"/>
-        <child link="right_gripper"/>
-    </joint>
-    <link name="right_gripper">
-        <visual>
-        <origin rpy="-3.1415 0 0" xyz="0 0 0"/>
-        <geometry>
-            <mesh filename="package://flex_gazebo/models/gripper/l_finger.dae"/>
-        </geometry>
-        </visual>
-        <collision>
-        <origin rpy="-3.1415 0 0" xyz="0 0 0"/>
-        <geometry>
-            <mesh filename="package://flex_gazebo/models/gripper/l_finger.dae"/>
-        </geometry>
-        </collision>
-    </link>
-    <joint name="right_tip_joint" type="fixed">
-        <parent link="right_gripper"/>
-        <child link="right_tip"/>
-    </joint>
-    <link name="right_tip">
-        <visual>
-        <origin rpy="-3.1415 0 0" xyz="0.09137 0.00495 0"/>
-        <geometry>
-            <mesh filename="package://flex_gazebo/models/gripper/l_finger_tip.dae"/>
-        </geometry>
-        </visual>
-        <collision>
-        <origin rpy="-3.1415 0 0" xyz="0.09137 0.00495 0"/>
-        <geometry>
-            <mesh filename="package://flex_gazebo/models/gripper/l_finger_tip.dae"/>
-        </geometry>
-        </collision>
-    </link>
-    <!--  Here we define another dummy joint. It is placed at the end of the tool, so we can then attach a frame at its TCP for control -->
-    <joint name="tool_tip_joint" type="fixed">
-        <parent link="gripper_pole" />
-        <child link = "tool_link_ee" />
-        <origin xyz="${tool_link_offset}" rpy="0 ${PI/2.0} 0" />
-    </joint>
-    <!--  The TCP frame is here defined -->
-    <link name="tool_link_ee"/>
+<robot xmlns:xacro="http://www.ros.org/wiki/xacro">
+  <xacro:include filename="$(find flex_gazebo)/urdf/gripper.gazebo.xacro" />
+  <xacro:include filename="$(find pr2_description)/urdf/gripper_v0/gripper.transmission.xacro" />
+  <xacro:property name="M_PI" value="3.1415926535897931" />
+  <xacro:property name="gripper_upper_angle" value="0.548" />
+  <xacro:property name="gripper_lower_angle" value="0.00" />
+  <xacro:property name="finger_damping"             value="0.02" />
+  <xacro:property name="gripper_damping"            value="10.0" />
+  <xacro:property name="finger_tip_damping"         value="0.001" />
+  <xacro:property name="finger_joint_effort_limit"  value="1000.0" />
+  <xacro:property name="finger_to_finger_tip_x"     value="0.09137" />
+  <xacro:property name="palm_to_finger_x"           value="0.07691" />
+  <xacro:macro name="pr2_finger_limits_v0">
+    <!-- limits on passive finger and finger top joints without
+         transmission are not enforced by safety controllers.
+         The lower/upper limits and are enforced in PR2 simulation and
+         effort and velocity limits are ignored. This is also needed because
+         these joints are declared revolute rather than continuous.-->
+    <limit effort="${finger_joint_effort_limit}" velocity="0.5"
+           lower="${gripper_lower_angle}" upper="${gripper_upper_angle}" />
+  </xacro:macro>
+  <xacro:macro name="pr2_finger_v0" params="prefix parent reflect">
+    <!-- Finger proximal digit -->
+    <joint name="${prefix}_l_finger_joint" type="revolute">
+      <axis xyz="0 0 1" />
+      <xacro:pr2_finger_limits_v0/>
+      <dynamics damping="${finger_damping}" />
+      <origin xyz="0.07691 0.01 0" rpy="0 0 0" />
+      <parent link="${parent}"/>
+      <child link="${prefix}_l_finger_link"/>
+    </joint>
+    <link name="${prefix}_l_finger_link">
+      <inertial>
+        <mass value="0.17126" />
+        <origin xyz="${0.03598} 0.01730 -0.00164" rpy="0 0 0" />
+        <inertia  ixx= "0.00007756198"
+                  ixy= "0.00000149095"
+                  ixz="-0.00000983385"
+                  iyy= "0.00019708305"
+                  iyz="-0.00000306125"
+                  izz= "0.00018105446" />
+      </inertial>
+      <visual>
+        <origin xyz="0 0 0" rpy="0 0 0" />
+        <geometry>
+          <mesh filename="package://pr2_description/meshes/gripper_v0/l_finger.dae" />
+        </geometry>
+        <material name="Grey" />
+      </visual>
+      <collision>
+        <origin xyz="0 0 0" rpy="0 0 0" />
+        <geometry>
+          <mesh filename="package://pr2_description/meshes/gripper_v0/l_finger.stl" />
+        </geometry>
+      </collision>
+    </link>
+    <!-- Finger proximal digit -->
+    <joint name="${prefix}_r_finger_joint" type="revolute">
+      <axis xyz="0 0 -1" />
+      <origin xyz="${palm_to_finger_x} -0.01 0" rpy="0 0 0" />
+      <xacro:pr2_finger_limits_v0/>
+      <dynamics damping="${finger_damping}" />
+      <mimic joint="${prefix}_l_finger_joint" multiplier="1" offset="0"/>
+      <parent link="${parent}"/>
+      <child link="${prefix}_r_finger_link"/>
+    </joint>
+    <link name="${prefix}_r_finger_link">
+      <inertial>
+        <mass value="0.17389" />
+        <origin xyz="${0.03576} -0.01736 -0.00095" rpy="0 0 0" />
+        <inertia  ixx= "0.00007738410"
+                  ixy="-0.00000209309"
+                  ixz="-0.00000836228"
+                  iyy= "0.00019847383"
+                  iyz= "0.00000246110"
+                  izz= "0.00018106988" />
+      </inertial>
+      <visual>
+        <origin xyz="0 0 0" rpy="${M_PI} 0 0" />
+        <geometry>
+          <mesh filename="package://pr2_description/meshes/gripper_v0/l_finger.dae" />
+        </geometry>
+        <material name="Grey" />
+      </visual>
+      <collision>
+        <origin xyz="0 0 0" rpy="${M_PI} 0 0" />
+        <geometry>
+          <mesh filename="package://pr2_description/meshes/gripper_v0/l_finger.stl" />
+        </geometry>
+      </collision>
+    </link>
+    <!-- Finger tip -->
+    <joint name="${prefix}_l_finger_tip_joint" type="revolute">
+      <axis xyz="0 0 -1" />
+      <origin xyz="${finger_to_finger_tip_x} 0.00495 0" rpy="0 0 0" />
+      <xacro:pr2_finger_limits_v0/>
+      <dynamics damping="${finger_tip_damping}" />
+      <mimic joint="${prefix}_l_finger_joint" multiplier="1" offset="0"/>
+      <parent link="${prefix}_l_finger_link"/>
+      <child link="${prefix}_l_finger_tip_link"/>
+    </joint>
+    <link name="${prefix}_l_finger_tip_link">
+      <inertial>
+        <mass value="0.04419" />
+        <origin xyz="0.00423 0.00284 0.0" rpy="0 0 0" />
+        <inertia  ixx="0.00000837047" ixy="0.00000583632" ixz="0.0"
+                  iyy="0.00000987067" iyz="0.0"
+                  izz="0.00001541768" />
+      </inertial>
+      <visual>
+        <origin xyz="0 0 0" rpy="0 0 0" />
+        <geometry>
+          <mesh filename="package://pr2_description/meshes/gripper_v0/l_finger_tip.dae" />
+        </geometry>
+        <material name="Green" />
+      </visual>
+      <collision>
+        <origin xyz="0 0 0" rpy="0 0 0" />
+        <geometry>
+          <mesh filename="package://pr2_description/meshes/gripper_v0/l_finger_tip.stl" />
+        </geometry>
+      </collision>
+    </link>
+    <!-- Finger tip -->
+    <joint name="${prefix}_r_finger_tip_joint" type="revolute">
+      <axis xyz="0 0 1" />
+      <origin xyz="${0.09137} ${-0.00495} 0" rpy="0 0 0" />
+      <xacro:pr2_finger_limits_v0/>
+      <dynamics damping="${finger_tip_damping}" />
+      <mimic joint="${prefix}_l_finger_joint" multiplier="1" offset="0"/>
+      <parent link="${prefix}_r_finger_link"/>
+      <child link="${prefix}_r_finger_tip_link"/>
+    </joint>
+    <link name="${prefix}_r_finger_tip_link">
+      <inertial>
+        <mass value="0.04419" />
+        <origin xyz="${0.00423} ${-0.00284} ${0.0}" rpy="0 0 0" />
+        <inertia  ixx="0.00000837047" ixy="-0.00000583632" ixz="0.0"
+                  iyy="0.00000987067" iyz="0.0"
+                  izz="0.00001541768" />
+      </inertial>
+      <visual>
+        <origin xyz="0 0 0" rpy="${M_PI} 0 0" />
+        <geometry>
+          <mesh filename="package://pr2_description/meshes/gripper_v0/l_finger_tip.dae"  />
+        </geometry>
+        <material name="Green" />
+      </visual>
+      <collision>
+        <origin xyz="0 0 0" rpy="${M_PI} 0 0" />
+        <geometry>
+          <mesh filename="package://pr2_description/meshes/gripper_v0/l_finger_tip.stl"  />
+        </geometry>
+      </collision>
+    </link>
+    <!-- extensions -->
+    <xacro:pr2_finger_gazebo_v0 prefix="${prefix}" reflect="${reflect}" />
+  </xacro:macro>
+  <xacro:macro name="pr2_gripper_v0" params="side reflect parent *origin gear_ratio screw_reduction theta0 phi0 t0 L0 h a b r">
+    <joint name="${side}_gripper_palm_joint" type="fixed">
+      <xacro:insert_block name="origin"/>
+      <parent link="${parent}"/>
+      <child link="${side}_gripper_palm_link"/>
+    </joint>
+    <link name="${side}_gripper_palm_link">
+      <inertial>
+        <mass value="0.58007" />
+        <origin xyz="0.06623 0.00053 -0.00119" rpy="0 0 0" />
+        <inertia  ixx="0.00035223921" ixy="-0.00001580476" ixz="-0.00000091750"
+                  iyy="0.00067741312" iyz="-0.00000059554"
+                  izz="0.00086563316" />
+      </inertial>
+      <visual>
+        <origin xyz="0 0 0" rpy="0 0 0" />
+        <geometry>
+          <mesh filename="package://pr2_description/meshes/gripper_v0/gripper_palm.dae"  />
+        </geometry>
+        <material name="Red" />
+      </visual>
+      <collision>
+        <origin xyz="0 0 0" rpy="0 0 0" />
+        <geometry>
+          <mesh filename="package://pr2_description/meshes/gripper_v0/gripper_palm.stl"  />
+        </geometry>
+      </collision>
+    </link>
+    <joint name="${side}_gripper_led_joint" type="fixed">
+      <!--  Need to check if we need a positive or negative Z term -->
+      <origin xyz="0.0513 0.0 .0244"/>
+      <parent link="${side}_gripper_palm_link"/>
+      <child link="${side}_gripper_led_frame"/>
+    </joint>
+    <link name="${side}_gripper_led_frame" />
+    <joint name="${side}_gripper_motor_accelerometer_joint" type="fixed">
+      <origin xyz="0 0 0" rpy="0 0 0" />
+      <parent link="${side}_gripper_palm_link"/>
+      <child link="${side}_gripper_motor_accelerometer_link"/>
+    </joint>
+    <link name="${side}_gripper_motor_accelerometer_link">
+      <inertial>
+        <mass value="0.001" />
+        <origin xyz="0 0 0" rpy="0 0 0" />
+        <inertia  ixx="0.001" ixy="0.0" ixz="0.0"
+                  iyy="0.001" iyz="0.0"
+                  izz="0.001" />
+      </inertial>
+      <visual>
+        <origin xyz="0 0 0" rpy="0 0 0" />
+        <geometry>
+          <box size="0.001 0.001 0.001" />
+        </geometry>
+      </visual>
+      <collision>
+        <origin xyz="0 0 0" rpy="0 0 0" />
+        <geometry>
+          <box size="0.001 0.001 0.001" />
+        </geometry>
+      </collision>
+    </link>
+    <joint name="${side}_gripper_tool_joint" type="fixed">
+      <origin xyz="0.18 0 0" rpy="0 0 0" />
+      <parent link="${side}_gripper_palm_link"/>
+      <child link="${side}_gripper_tool_frame"/>
+    </joint>
+    <link name="${side}_gripper_tool_frame"/>
+    <!-- actuated motor screw joint -->
+    <link name="${side}_gripper_motor_slider_link">
+      <inertial>
+        <mass value="0.01" />
+        <origin xyz="0 0 0" rpy="0 0 0" />
+        <inertia  ixx="0.001" ixy="0.0" ixz="0.0"
+                  iyy="0.001" iyz="0.0"
+                  izz="0.001" />
+      </inertial>
+      <!-- for debugging only
+      <visual>
+        <origin xyz="0 0 0" rpy="1.5708 0 0" />
+        <geometry>
+          <cylinder length="0.002" radius="0.025"/>
+        </geometry>
+      </visual>
+      <collision>
+        <origin xyz="0 0 0" rpy="1.5708 0 0" />
+        <geometry>
+          <cylinder length="0.002" radius="0.025"/>
+        </geometry>
+      </collision>
+      -->
+    </link>
+    <joint name="${side}_gripper_motor_slider_joint" type="prismatic">
+      <origin xyz="${finger_to_finger_tip_x+palm_to_finger_x} 0 0" rpy="0 0 0" />
+      <axis xyz="1 0 0"/>
+      <parent link="${side}_gripper_palm_link"/>
+      <child link="${side}_gripper_motor_slider_link"/>
+      <limit effort="1000.0" velocity="0.2" lower="-0.1" upper="0.1" />
+    </joint>
+    <link name="${side}_gripper_motor_screw_link">
+      <inertial>
+        <mass value="0.01" />
+        <origin xyz="0 0 0" rpy="0 0 0" />
+        <inertia  ixx="0.0001" ixy="0.0" ixz="0.0"
+                  iyy="0.0001" iyz="0.0"
+                  izz="0.0001" />
+      </inertial>
+      <!-- for debugging only
+      <visual>
+        <origin xyz="0 0 0" rpy="0 0 0" />
+        <geometry>
+          <box size="0.05 0.001 0.05" />
+        </geometry>
+      </visual>
+      <collision>
+        <origin xyz="0 0 0" rpy="0 0 0" />
+        <geometry>
+          <box size="0.05 0.001 0.05" />
+        </geometry>
+      </collision>
+      -->
+    </link>
+    <joint name="${side}_gripper_motor_screw_joint" type="continuous">
+      <origin xyz="0.0 0 0" rpy="0 0 0" />
+      <axis xyz="0 1 0"/>
+      <parent link="${side}_gripper_motor_slider_link"/>
+      <child link="${side}_gripper_motor_screw_link"/>
+      <dynamics damping="0.0001" />
+    </joint>
+    <!-- pr2 fingers macro -->
+    <xacro:pr2_finger_v0 prefix="${side}_gripper" reflect="${reflect}" parent="${side}_gripper_palm_link" />
+    <!-- fictitous joint that represents the gripper gap -->
+    <!-- effort is the linear force at the gripper gap
+         velocity limit is the linear velocity limit at the gripper gap
+         try and introduce a very stiff spring
+         The velocity limits are alpha tested.
+         The effort limits are somewhat inflated.
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
File: flex_gazebo/urdf/robot.urdf.xacro (robot description, xacro)
@@ -8,4 +8,7 @@
   <xacro:include filename="$(find realsense2_description)/urdf/_d435.urdf.xacro" />
   <xacro:include filename="$(find flex_gazebo)/urdf/camera/camera.gazebo.xacro" />
+  <!-- end-effector -->
+  <xacro:arg name="ee" default="pr2"/>
+  <xacro:property name="ee" value="$(arg ee)"/>
   <!-- iiwa params-->
   <xacro:arg name="hardware_interface" default="PositionJointInterface"/>
@@ -29,4 +32,36 @@
   </xacro:sensor_d435>
   <xacro:my_camera name="$(arg camera_name)"/>
+  <xacro:if value="${ee == 'sdh'}">
+    <xacro:include filename="$(find schunk_description)/urdf/sdh/sdh.urdf.xacro" />
+    <xacro:arg name="endeffector_name" default="sdh"/>
+    <xacro:arg name="endeffector_origin_xyz" default="0 0 0"/>
+    <xacro:arg name="endeffector_origin_rpy" default="0 0 0"/>
+    <xacro:schunk_sdh parent="iiwa_link_ee" name="$(arg endeffector_name)">
+      <origin xyz="$(arg endeffector_origin_xyz)" rpy="$(arg endeffector_origin_rpy)" />
+    </xacro:schunk_sdh>
+  </xacro:if>
+  <xacro:if value="${ee == 'pr2'}" >
+    <xacro:include filename="$(find flex_gazebo)/urdf/gripper.urdf.xacro" />
+    <!--
+    <xacro:include filename="$(find pr2_description)/urdf/materials.urdf.xacro" />
+    -->
+    <xacro:include filename="$(find pr2_description)/gazebo/gazebo.urdf.xacro" />
+    <xacro:include filename="$(find pr2_description)/urdf/common.xacro" />
+    <xacro:arg name="endeffector_origin_xyz" default="0 0 -0.03576"/>
+    <xacro:arg name="endeffector_origin_rpy" default="0 -${M_PI/2} 0"/>
+    <xacro:pr2_gripper_v0 reflect="-1.0" side="r" parent="iiwa_link_ee"
+                          screw_reduction="${4.0/1000.0}"
+                          gear_ratio="${(729.0/25.0)*(22.0/16.0)}"
+                          theta0="${3.6029*M_PI/180.0}"
+                          phi0="${29.7089*M_PI/180.0}"
+                          t0="${-0.1914/1000.0}"
+                          L0="${37.5528/1000.0}"
+                          h="${0.0/1000.0}"
+                          a="${68.3698/1000.0}"
+                          b="${43.3849/1000.0}"
+                          r="${91.5/1000.0}">
+      <origin xyz="$(arg endeffector_origin_xyz)" rpy="$(arg endeffector_origin_rpy)" />
+    </xacro:pr2_gripper_v0>
+  </xacro:if>
 </robot>
 <!-- This does not belong here! -->
