Commit message: We can now give object arguments to the enviroment.launch file

File: flex_gazebo/urdf/world.urdf.xacro (robot description, xacro)
@@ -1,15 +1,15 @@
 <?xml version="1.0"?>
 <robot name="world" xmlns:xacro="http://www.ros.org/wiki/xacro">
-  <xacro:arg name="dimensions" default="3d"/>
+  <xacro:arg name="object_name" default="truss"/>
+  <xacro:arg name="object_dimension" default="3d"/>
+  <xacro:arg name="object_origin_xyz" default="-0.2 0.4 0.26"/>
+  <xacro:arg name="object_origin_rpy" default="0.0 0.0 0.0"/>
   <!-- import the tomato -->
-  <xacro:include filename="$(find flex_gazebo)/urdf/truss/$(arg dimensions)/truss.xacro"/>
-  <!-- tomato params-->
-  <xacro:arg name="truss_origin_xyz" default="-0.2 0.4 0.26"/>
-  <xacro:arg name="truss_origin_rpy" default="0.0 0.0 $(arg tomato_angle)"/>
+  <xacro:include filename="$(find flex_gazebo)/urdf/$(arg object_name)/$(arg object_dimension)/$(arg object_name).xacro"/>
   <!-- Fix to world just for testing -->
   <link name="world"/>
   <!-- tomato -->
   <xacro:truss>
-    <origin xyz="$(arg truss_origin_xyz)" rpy="$(arg truss_origin_rpy)" />
+    <origin xyz="$(arg object_origin_xyz)" rpy="$(arg object_origin_rpy)" />
   </xacro:truss>
 </robot>
