Commit message: flex_gazebo.launch working with px150, next step is moveit.

File: flex_gazebo/urdf/iiwa_tool.urdf.xacro (robot description, xacro)
@@ -4,7 +4,7 @@
   <xacro:macro name="endeffector">
     <!-- End-effector params -->
-    <property name="tool_mass" value="0.200" />
-    <property name="tool_joint_offset" value="0.00 0.00 0.00" />
-    <property name="tool_link_offset" value="0.2 0.00 0" />
+    <xacro:property name="tool_mass" value="0.200" />
+    <xacro:property name="tool_joint_offset" value="0.00 0.00 0.00" />
+    <xacro:property name="tool_link_offset" value="0.2 0.00 0" />
     <!--  Here we define a dummy joint between the tip of the iiwa7 and the base of the tool.
     There is no offset between the two, that means the tool is attached at the robot flange. -->

File: flex_gazebo/urdf/robot.urdf.xacro (robot description, xacro)
@@ -1,37 +1,67 @@
 <?xml version="1.0"?>
 <robot name="iiwa7" xmlns:xacro="http://www.ros.org/wiki/xacro">
-  <!-- Import Rviz colors -->
-  <xacro:include filename="$(find iiwa_description)/urdf/materials.xacro" />
-  <!--Import the lbr iiwa macro -->
-  <xacro:include filename="$(find iiwa_description)/urdf/iiwa7.xacro"/>
+  <!-- General parameters -->
+  <xacro:arg name="use_sdh" default="false"/>
+  <xacro:arg name="use_iiwa" default="false"/>
+  <xacro:arg name="use_interbotix" default="false"/>
+  <!-- iiwa params-->
+  <xacro:arg name="hardware_interface" default="PositionJointInterface"/>
+  <xacro:arg name="robot_name" default="iiwa"/>
+  <xacro:arg name="robot_model" default="iiwa7"/>
+  <!-- camera params-->
+  <xacro:arg name="camera_name" default="rs_d435"/>
+  <xacro:arg name="camera_sim" default="true"/>
+  <xacro:arg name="camera_origin_xyz" default="0 0.6 1.2"/>
+  <xacro:arg name="camera_origin_rpy" default="3.1415 1.57 -1.57"/>
+  <xacro:arg name="iiwa_origin_xyz" default="0.0 0.0 0.0"/>
+  <xacro:arg name="iiwa_origin_rpy" default="0.0 0.0 0.0"/>
+  <xacro:arg name="interbotix_origin_xyz" default="0.0 0.0 0.26"/>
+  <xacro:arg name="interbotix_origin_rpy" default="0.0 0.0 ${3.1415 / 2}"/>
+    <!-- end-effector params-->
+  <xacro:arg name="endeffector_name" default="sdh"/>
+  <xacro:arg name="endeffector_origin_xyz" default="0 0 0"/>
+  <xacro:arg name="endeffector_origin_rpy" default="0 0 0"/>
+  <xacro:arg name="use_nominal_extrinsics" default="$(arg camera_sim)"/>
   <!-- import the camera -->
   <xacro:include filename="$(find realsense2_description)/urdf/_d435.urdf.xacro" />
   <xacro:include filename="$(find flex_gazebo)/urdf/camera/camera.gazebo.xacro" />
-  <!-- import the end-effector -->
-  <xacro:include filename="$(find flex_gazebo)/urdf/iiwa_tool.urdf.xacro" />
-  <!-- iiwa params-->
-  <xacro:arg name="hardware_interface" default="PositionJointInterface"/>
-  <xacro:arg name="robot_name" default="iiwa"/>
-  <xacro:arg name="origin_xyz" default="0 0 0"/>
-  <xacro:arg name="origin_rpy" default="0 0 0"/>
-  <!-- camera params-->
-  <xacro:arg name="camera_name" default="camera"/>
-  <xacro:arg name="camera_origin_xyz" default="0 0.6 1.2"/>
-  <xacro:arg name="camera_origin_rpy" default="3.1415 1.57 -1.57"/>
-  <xacro:arg name="use_nominal_extrinsics" default="true"/>
-  <!-- Fix to world just for testing -->
+  <!-- Fix to world -->
   <link name="world"/>
   <!--iiwa -->
-  <xacro:iiwa7 hardware_interface="$(arg hardware_interface)" robot_name="$(arg robot_name)" parent="world">
-    <origin xyz="$(arg origin_xyz)" rpy="$(arg origin_rpy)" />
-  </xacro:iiwa7>
+  <xacro:if value="$(arg use_iiwa)">
+    <!-- Import Rviz colors -->
+    <xacro:include filename="$(find iiwa_description)/urdf/materials.xacro" />
+    <!--Import the lbr iiwa macro -->
+    <xacro:include filename="$(find iiwa_description)/urdf/iiwa7.xacro"/>
+    <xacro:iiwa7 hardware_interface="$(arg hardware_interface)" robot_name="$(arg robot_name)" parent="world">
+      <origin xyz="$(arg iiwa_origin_xyz)" rpy="$(arg iiwa_origin_rpy)" />
+    </xacro:iiwa7>
+    <!-- end-effector -->
+    <xacro:if value="$(arg use_sdh)">
+      <!-- import the end-effector -->
+      <xacro:include filename="$(find schunk_description)/urdf/sdh/sdh.urdf.xacro" />
+      <xacro:schunk_sdh parent="iiwa_link_ee" name="$(arg endeffector_name)">
+        <origin xyz="$(arg endeffector_origin_xyz)" rpy="$(arg endeffector_origin_rpy)" />
+      </xacro:schunk_sdh>
+    </xacro:if>
+  </xacro:if>
+  <!--interbotix -->
+  <xacro:if value="$(arg use_interbotix)">
+    <joint name="fixed" type="fixed">
+      <parent link="world"/>
+      <child link="$(arg robot_name)/base_link"/>
+      <origin xyz="$(arg interbotix_origin_xyz)" rpy="$(arg interbotix_origin_rpy)"/>
+    </joint>
+    <xacro:include filename="$(find flex_gazebo)/urdf/px150.xacro"/>
+    <xacro:px150>
+    </xacro:px150>
+  </xacro:if>
   <!-- camera -->
   <xacro:sensor_d435 parent="world" name="$(arg camera_name)" use_nominal_extrinsics="$(arg use_nominal_extrinsics)">
     <origin xyz="$(arg camera_origin_xyz)" rpy="$(arg camera_origin_rpy)" />
   </xacro:sensor_d435>
-  <xacro:my_camera name="$(arg camera_name)"/>
-  <!-- end-effector -->
-  <xacro:endeffector>
-  </xacro:endeffector>
+  <xacro:if value="$(arg camera_sim)">
+    <xacro:my_camera name="$(arg camera_name)"/>
+  </xacro:if>
 </robot>
 <!-- This does not belong here! -->

File: flex_gazebo/urdf/robot_old.urdf.xacro (robot description, xacro)
@@ -8,7 +8,6 @@
   <xacro:include filename="$(find realsense2_description)/urdf/_d435.urdf.xacro" />
   <xacro:include filename="$(find flex_gazebo)/urdf/camera/camera.gazebo.xacro" />
-  deve
   <!-- import the end-effector -->
-  <xacro:include filename="$(find schunk_description)/urdf/sdh/sdh.urdf.xacro" />
+  <xacro:include filename="$(find flex_gazebo)/urdf/iiwa_tool.urdf.xacro" />
   <!-- iiwa params-->
   <xacro:arg name="hardware_interface" default="PositionJointInterface"/>
@@ -17,13 +16,8 @@
   <xacro:arg name="origin_rpy" default="0 0 0"/>
   <!-- camera params-->
-  <xacro:arg name="camera_name" default="rs_d435"/>
-  <xacro:arg name="camera_sim" default="true"/>
+  <xacro:arg name="camera_name" default="camera"/>
   <xacro:arg name="camera_origin_xyz" default="0 0.6 1.2"/>
   <xacro:arg name="camera_origin_rpy" default="3.1415 1.57 -1.57"/>
-    <!-- end-effector params-->
-  <xacro:arg name="endeffector_name" default="sdh"/>
-  <xacro:arg name="endeffector_origin_xyz" default="0 0 0"/>
-  <xacro:arg name="endeffector_origin_rpy" default="0 0 0"/>
-  <xacro:arg name="use_nominal_extrinsics" default="$(arg camera_sim)"/>
+  <xacro:arg name="use_nominal_extrinsics" default="true"/>
   <!-- Fix to world just for testing -->
   <link name="world"/>
@@ -36,11 +30,8 @@
     <origin xyz="$(arg camera_origin_xyz)" rpy="$(arg camera_origin_rpy)" />
   </xacro:sensor_d435>
-  <xacro:if value="$(arg camera_sim)">
-    <xacro:my_camera name="$(arg camera_name)"/>
-  </xacro:if>
+  <xacro:my_camera name="$(arg camera_name)"/>
   <!-- end-effector -->
-  <xacro:schunk_sdh parent="iiwa_link_ee" name="$(arg endeffector_name)">
-      <origin xyz="$(arg endeffector_origin_xyz)" rpy="$(arg endeffector_origin_rpy)" />
-  </xacro:schunk_sdh>
+  <xacro:endeffector>
+  </xacro:endeffector>
 </robot>
 <!-- This does not belong here! -->
