Commit message: No longer showing the tomato truss in rviz

File: flex_gazebo/urdf/camera.urdf.xacro (robot description, xacro)
@@ -3,5 +3,5 @@
   <!-- import the camera -->
   <xacro:include filename="$(find realsense2_description)/urdf/_d435.urdf.xacro" />
-  <!-- <xacro:include filename="$(find realsense_gazebo_plugin)/urdf/realsense-RS200.macro.xacro" /> -->
+  <!-- camera params-->
   <xacro:arg name="camera_name" default="camera"/>
   <xacro:arg name="camera_origin_xyz" default="0 0.6 1.2"/>
@@ -10,11 +10,12 @@
   <!-- Fix to world just for testing -->
   <link name="world"/>
+  <!-- camera -->
   <xacro:sensor_d435 parent="world" name="$(arg camera_name)" use_nominal_extrinsics="$(arg use_nominal_extrinsics)">
     <origin xyz="$(arg camera_origin_xyz)" rpy="$(arg camera_origin_rpy)" />
   </xacro:sensor_d435>
-  <!--
-  <xacro:realsense-rs200 parent="world" prefix="$(arg camera_name)">
-    <origin xyz="$(arg camera_origin_xyz)" rpy="$(arg camera_origin_rpy)" />
-  </xacro:realsense-rs200>
-  -->
 </robot>
+<!-- This does not belong here! -->
+<!--
+<robot name="realsense2_camera" xmlns:xacro="http://ros.org/wiki/xacro">
+</robot>
+ -->

File: flex_gazebo/urdf/robot.urdf.xacro (robot description, xacro)
@@ -7,6 +7,4 @@
   <!-- import the camera -->
   <xacro:include filename="$(find realsense2_description)/urdf/_d435.urdf.xacro" />
-  <!-- import the tomato -->
-  <xacro:include filename="$(find flex_gazebo)/urdf/tomato.xacro" />
   <!-- iiwa params-->
   <xacro:arg name="hardware_interface" default="PositionJointInterface"/>
@@ -19,7 +17,4 @@
   <xacro:arg name="camera_origin_rpy" default="3.1415 1.57 -1.57"/>
   <xacro:arg name="use_nominal_extrinsics" default="true"/>
-  <!-- tomato params-->
-  <xacro:arg name="tomato_origin_xyz" default="-0.2 0.4 0.26"/>
-  <xacro:arg name="tomato_origin_rpy" default="0 0 0.3"/>
   <!-- Fix to world just for testing -->
   <link name="world"/>
@@ -32,8 +27,4 @@
     <origin xyz="$(arg camera_origin_xyz)" rpy="$(arg camera_origin_rpy)" />
   </xacro:sensor_d435>
-  <!-- tomato -->
-  <xacro:tomato_2d>
-    <origin xyz="$(arg tomato_origin_xyz)" rpy="$(arg tomato_origin_rpy)" />
-  </xacro:tomato_2d>
 </robot>
 <!-- This does not belong here! -->

Commit message: Now added camera to gezebo based on correct frames, robot moves to the right position

File: flex_gazebo/urdf/camera.urdf.xacro (robot description, xacro)
@@ -3,4 +3,5 @@
   <!-- import the camera -->
   <xacro:include filename="$(find realsense2_description)/urdf/_d435.urdf.xacro" />
+  <xacro:include filename="$(find flex_gazebo)/urdf/camera/camera.gazebo.xacro" />
   <!-- camera params-->
   <xacro:arg name="camera_name" default="camera"/>
@@ -14,4 +15,5 @@
     <origin xyz="$(arg camera_origin_xyz)" rpy="$(arg camera_origin_rpy)" />
   </xacro:sensor_d435>
+  <xacro:my_camera name="$(arg camera_name)"/>
 </robot>
 <!-- This does not belong here! -->

File: flex_gazebo/urdf/robot.urdf.xacro (robot description, xacro)
@@ -7,4 +7,5 @@
   <!-- import the camera -->
   <xacro:include filename="$(find realsense2_description)/urdf/_d435.urdf.xacro" />
+  <xacro:include filename="$(find flex_gazebo)/urdf/camera/camera.gazebo.xacro" />
   <!-- iiwa params-->
   <xacro:arg name="hardware_interface" default="PositionJointInterface"/>
@@ -27,4 +28,5 @@
     <origin xyz="$(arg camera_origin_xyz)" rpy="$(arg camera_origin_rpy)" />
   </xacro:sensor_d435>
+  <xacro:my_camera name="$(arg camera_name)"/>
 </robot>
 <!-- This does not belong here! -->

File: flex_gazebo/urdf/world.urdf.xacro (robot description, xacro)
@@ -3,5 +3,4 @@
   <!-- import the tomato -->
   <xacro:include filename="$(find flex_gazebo)/urdf/tomato/3d/truss.xacro"/>
-  <!-- <xacro:include filename="$(find realsense_gazebo_plugin)/urdf/realsense-RS200.macro.xacro" /> -->
   <!-- tomato params-->
   <xacro:arg name="truss_origin_xyz" default="-0.2 0.4 0.26"/>
@@ -13,8 +12,3 @@
     <origin xyz="$(arg truss_origin_xyz)" rpy="$(arg truss_origin_rpy)" />
   </xacro:truss>
-  <!--
-  <xacro:realsense-rs200 parent="world" prefix="$(arg camera_name)">
-    <origin xyz="$(arg camera_origin_xyz)" rpy="$(arg camera_origin_rpy)" />
-  </xacro:realsense-rs200>
-  -->
 </robot>

Commit message: Modified file for testing camera + marker set up

File: flex_gazebo/urdf/camera.urdf.xacro (robot description, xacro)
@@ -4,9 +4,14 @@
   <xacro:include filename="$(find realsense2_description)/urdf/_d435.urdf.xacro" />
   <xacro:include filename="$(find flex_gazebo)/urdf/camera/camera.gazebo.xacro" />
+  <!-- Impoprt the aruco marker -->
+  <xacro:include filename="$(find flex_gazebo)/urdf/marker/marker.xacro"/>
   <!-- camera params-->
   <xacro:arg name="camera_name" default="camera"/>
-  <xacro:arg name="camera_origin_xyz" default="0 0.6 1.2"/>
+  <xacro:arg name="camera_origin_xyz" default="0 0 0.5"/>
   <xacro:arg name="camera_origin_rpy" default="3.1415 1.57 -1.57"/>
   <xacro:arg name="use_nominal_extrinsics" default="true"/>
+  <!-- marker params -->
+  <xacro:arg name="marker_origin_xyz" default="0 0 0"/>
+  <xacro:arg name="marker_origin_rpy" default="0 0 0"/>
   <!-- Fix to world just for testing -->
   <link name="world"/>
@@ -16,4 +21,7 @@
   </xacro:sensor_d435>
   <xacro:my_camera name="$(arg camera_name)"/>
+  <xacro:marker parent_link="world" size="0.04" ID ="26" >
+    <origin xyz="$(arg marker_origin_xyz)" rpy="$(arg marker_origin_rpy)" />
+  </xacro:marker>
 </robot>
 <!-- This does not belong here! -->

File: flex_gazebo/urdf/marker/marker.xacro (robot description, xacro)
@@ -3,5 +3,5 @@
 <xacro:include filename="$(find flex_gazebo)/urdf/marker/marker.gazebo.xacro" />
   <xacro:macro name="marker" params="parent_link size ID *origin">
-    <xacro:property name = "xyz" value="-0.02 0 0.036"/>
+    <xacro:property name = "xyz" value="0 0 0"/>
     <joint name="marker__${ID}_joint" type="fixed">
       <xacro:insert_block name="origin" />

File: flex_gazebo/urdf/robot.urdf.xacro (robot description, xacro)
@@ -40,5 +40,5 @@
   <xacro:arg name="endeffector_origin_rpy" default="0 0 0"/>
   <xacro:arg name="use_nominal_extrinsics" default="$(arg camera_sim)"/>
-  <xacro:arg name="marker_origin_xyz" default="0 0 0.05"/>
+  <xacro:arg name="marker_origin_xyz" default="-0.02 0 0.036"/>
   <xacro:arg name="marker_origin_rpy" default="0 0 0"/>
   <!-- Fix to world -->
