Commit message: Added 3D tomato model

File: flex_gazebo/urdf/tomato/2d/tomato.xacro (robot description, xacro)
@@ -2,6 +2,10 @@
 <robot xmlns:xacro="http://www.ros.org/wiki/xacro">
   <!-- Import all Gazebo-customization elements, including Gazebo colors -->
-  <xacro:include filename="$(find flex_gazebo)/urdf/tomato.gazebo.xacro" />
+  <xacro:include filename="$(find flex_gazebo)/urdf/tomato/2d/tomato.gazebo.xacro" />
   <xacro:macro name="tomato_2d" params="*origin">
+    <xacro:property name="height" value="0.01" />
+    <xacro:property name="width" value="0.18" />
+    <xacro:property name="length" value="0.15" />
+    <xacro:property name="size" value="${length} ${width} ${height}" />
     <joint name="tomato_joint" type="floating">
       <xacro:insert_block name="origin" />
@@ -13,5 +17,5 @@
         <origin xyz="0 0 0" rpy="0 0 0"/>
         <geometry>
-          <box size = "0.15 0.18 0.001" />
+          <box size = "${size}" />
         </geometry>
       </collision>
@@ -19,11 +23,12 @@
         <origin xyz="0 0 0" rpy="0 0 0"/>
         <geometry>
-          <box size = "0.15 0.18 0.001" />
+          <box size = "${size}" />
         </geometry>
         <material name="Blue"/>
       </visual>
       <inertial>
-        <origin xyz="0 0 0" rpy="0 0 0"/>
-        <mass value="1"/>
+        <origin xyz="${length/2} ${width/2} ${height/2}" rpy="0 0 0"/>
+        <parent link="world"/>
+        <mass value="10"/>
         <inertia
 	         ixx="1.0" ixy="0.0" ixz="0.0"

File: flex_gazebo/urdf/world.urdf.xacro (robot description, xacro)
@@ -2,15 +2,15 @@
 <robot name="world" xmlns:xacro="http://www.ros.org/wiki/xacro">
   <!-- import the tomato -->
-  <xacro:include filename="$(find flex_gazebo)/urdf/tomato.xacro" />
+  <xacro:include filename="$(find flex_gazebo)/urdf/tomato/3d/truss.xacro"/>
   <!-- <xacro:include filename="$(find realsense_gazebo_plugin)/urdf/realsense-RS200.macro.xacro" /> -->
   <!-- tomato params-->
-  <xacro:arg name="tomato_origin_xyz" default="-0.2 0.4 0.26"/>
-  <xacro:arg name="tomato_origin_rpy" default="0.0 0.0 $(arg tomato_angle)"/>
+  <xacro:arg name="truss_origin_xyz" default="-0.2 0.4 0.26"/>
+  <xacro:arg name="truss_origin_rpy" default="0.0 0.0 $(arg tomato_angle)"/>
   <!-- Fix to world just for testing -->
   <link name="world"/>
   <!-- tomato -->
-  <xacro:tomato_2d>
-    <origin xyz="$(arg tomato_origin_xyz)" rpy="$(arg tomato_origin_rpy)" />
-  </xacro:tomato_2d>
+  <xacro:truss>
+    <origin xyz="$(arg truss_origin_xyz)" rpy="$(arg truss_origin_rpy)" />
+  </xacro:truss>
   <!--
   <xacro:realsense-rs200 parent="world" prefix="$(arg camera_name)">
