Commit message: Fixed tomato to the peduncle

File: flex_gazebo/urdf/tomato/3d/tomato.xacro (robot description, xacro)
@@ -5,5 +5,5 @@
   <xacro:macro name="tomato" params="tomato_name radius parent_link *origin">
     <xacro:property name="distance" value="0.1" />
-    <joint name="tomato_joint${tomato_name}" type="floating">
+    <joint name="tomato_joint${tomato_name}" type="fixed">
       <xacro:insert_block name="origin" />
       <parent link="${parent_link}"/>
