Commit message: Fixed mistake in pose transform, we can now easily change between 2D and 3D tomatoes

File: flex_gazebo/urdf/truss/2d/truss.xacro (robot description, xacro)
@@ -2,7 +2,7 @@
 <robot xmlns:xacro="http://www.ros.org/wiki/xacro">
   <!-- Import all Gazebo-customization elements, including Gazebo colors -->
-  <xacro:include filename="$(find flex_gazebo)/urdf/tomato/2d/tomato.gazebo.xacro" />
-  <xacro:macro name="tomato_2d" params="*origin">
-    <xacro:property name="height" value="0.01" />
+  <xacro:include filename="$(find flex_gazebo)/urdf/truss/2d/tomato.gazebo.xacro" />
+  <xacro:macro name="truss" params="*origin">
+    <xacro:property name="height" value="0.10" />
     <xacro:property name="width" value="0.18" />
     <xacro:property name="length" value="0.15" />

File: flex_gazebo/urdf/truss/3d/peduncle.xacro (robot description, xacro)
@@ -1,5 +1,5 @@
 <?xml version="1.0"?>
 <robot xmlns:xacro="http://www.ros.org/wiki/xacro">
-  <xacro:include filename="$(find flex_gazebo)/urdf/tomato/3d/peduncle.gazebo.xacro" />
+  <xacro:include filename="$(find flex_gazebo)/urdf/truss/3d/peduncle.gazebo.xacro" />
   <xacro:macro name="peduncle" params="peduncle_length peduncle_radius parent_link">
     <xacro:property name = "PI" value="3.14159"/>

File: flex_gazebo/urdf/truss/3d/tomato.xacro (robot description, xacro)
@@ -2,5 +2,5 @@
 <robot xmlns:xacro="http://www.ros.org/wiki/xacro">
   <!-- Import all Gazebo-customization elements, including Gazebo colors -->
-  <xacro:include filename="$(find flex_gazebo)/urdf/tomato/3d/tomato.gazebo.xacro" />
+  <xacro:include filename="$(find flex_gazebo)/urdf/truss/3d/tomato.gazebo.xacro" />
   <xacro:macro name="tomato" params="tomato_name radius parent_link *origin">
     <xacro:property name="distance" value="0.1" />

File: flex_gazebo/urdf/truss/3d/truss.xacro (robot description, xacro)
@@ -2,6 +2,6 @@
 <robot xmlns:xacro="http://www.ros.org/wiki/xacro">
   <!-- Import all Gazebo-customization elements, including Gazebo colors -->
-  <xacro:include filename="$(find flex_gazebo)/urdf/tomato/3d/tomato.xacro"/>
-  <xacro:include filename="$(find flex_gazebo)/urdf/tomato/3d/peduncle.xacro"/>
+  <xacro:include filename="$(find flex_gazebo)/urdf/truss/3d/tomato.xacro"/>
+  <xacro:include filename="$(find flex_gazebo)/urdf/truss/3d/peduncle.xacro"/>
   <xacro:macro name="truss" params="*origin">
     <xacro:property name="tomato_radius" value="0.05" />

File: flex_gazebo/urdf/world.urdf.xacro (robot description, xacro)
@@ -1,6 +1,7 @@
 <?xml version="1.0"?>
 <robot name="world" xmlns:xacro="http://www.ros.org/wiki/xacro">
+  <xacro:arg name="dimensions" default="3d"/>
   <!-- import the tomato -->
-  <xacro:include filename="$(find flex_gazebo)/urdf/tomato/3d/truss.xacro"/>
+  <xacro:include filename="$(find flex_gazebo)/urdf/truss/$(arg dimensions)/truss.xacro"/>
   <!-- tomato params-->
   <xacro:arg name="truss_origin_xyz" default="-0.2 0.4 0.26"/>
