Commit message: grasp almost working, controllers behave strange, tomato slips.

File: flex_gazebo/urdf/truss/3d/peduncle.xacro (robot description, xacro)
@@ -3,5 +3,7 @@
   <xacro:include filename="$(find flex_gazebo)/urdf/truss/3d/peduncle.gazebo.xacro" />
   <xacro:macro name="peduncle" params="peduncle_length peduncle_radius parent_link">
-    <xacro:property name = "PI" value="3.14159"/>
+    <xacro:property name = "rho" value="1000"/> <!-- [kg/m^3]-->
+    <xacro:property name = "volume" value="${pi*peduncle_length*peduncle_radius**2}"/> <!-- [m^3]-->
+    <xacro:property name = "mass" value="${rho * volume}"/> <!-- [kg]-->
     <joint name="truss_joint" type="floating">
       <xacro:insert_block name="origin" />
@@ -12,5 +14,5 @@
       <collision>
         <!-- origin is in the center of the cylinder-->
-        <origin xyz="0 0 0" rpy="${PI/2} 0 0"/>
+        <origin xyz="0 0 0" rpy="${pi/2} 0 0"/>
         <geometry>
           <cylinder radius="${peduncle_radius}" length="${peduncle_length}"/>
@@ -18,5 +20,5 @@
       </collision>
       <visual>
-        <origin xyz="0 0 0" rpy="${PI/2} 0 0"/>
+        <origin xyz="0 0 0" rpy="${pi/2} 0 0"/>
         <geometry>
           <cylinder radius="${peduncle_radius}" length="${peduncle_length}"/>
@@ -26,9 +28,9 @@
       <inertial>
         <origin xyz="0 0 0" rpy="0 0 0"/>
-        <mass value="10"/>
+        <mass value="${mass}"/>
         <inertia
-           ixx="1.0" ixy="0.0" ixz="0.0"
-           iyy="1.0" iyz="0.0"
-           izz="1.0"/>
+           ixx="${1/12*mass*peduncle_length**2}" ixy="0.0" ixz="0.0"
+           iyy="${1/12*mass*peduncle_length**2}" iyz="0.0"
+           izz="${1/2*mass*peduncle_radius**2}"/>
        </inertial>
      </link>

File: flex_gazebo/urdf/truss/3d/tomato.xacro (robot description, xacro)
@@ -4,5 +4,7 @@
   <xacro:include filename="$(find flex_gazebo)/urdf/truss/3d/tomato.gazebo.xacro" />
   <xacro:macro name="tomato" params="tomato_name radius parent_link *origin">
-    <xacro:property name="distance" value="0.1" />
+    <xacro:property name = "rho" value="1000"/> <!-- [kg/m^3]-->
+    <xacro:property name = "V" value="${4/3*pi*radius**3}"/> <!-- [m^3]-->
+    <xacro:property name = "mass" value="${rho * V}"/> <!-- [kg]-->
     <joint name="tomato_joint${tomato_name}" type="fixed">
       <xacro:insert_block name="origin" />
@@ -26,9 +28,9 @@
       <inertial>
         <origin xyz="0 0 0" rpy="0 0 0"/>
-        <mass value="10"/>
+        <mass value="${mass}"/>
         <inertia
-	         ixx="1.0" ixy="0.0" ixz="0.0"
-           iyy="1.0" iyz="0.0"
-           izz="1.0"/>
+	         ixx="${2/5*mass*radius**2}" ixy="0.0" ixz="0.0"
+           iyy="${2/5*mass*radius**2}" iyz="0.0"
+           izz="${2/5*mass*radius**2}"/>
        </inertial>
      </link>

Commit message: Modified truss weight and pose transform, picking up tomatoes!

File: flex_gazebo/urdf/truss/3d/peduncle.xacro (robot description, xacro)
@@ -3,5 +3,5 @@
   <xacro:include filename="$(find flex_gazebo)/urdf/truss/3d/peduncle.gazebo.xacro" />
   <xacro:macro name="peduncle" params="peduncle_length peduncle_radius parent_link">
-    <xacro:property name = "rho" value="1000"/> <!-- [kg/m^3]-->
+    <xacro:property name = "rho" value="1"/> <!-- [kg/m^3]-->
     <xacro:property name = "volume" value="${pi*peduncle_length*peduncle_radius**2}"/> <!-- [m^3]-->
     <xacro:property name = "mass" value="${rho * volume}"/> <!-- [kg]-->

File: flex_gazebo/urdf/truss/3d/tomato.xacro (robot description, xacro)
@@ -4,5 +4,5 @@
   <xacro:include filename="$(find flex_gazebo)/urdf/truss/3d/tomato.gazebo.xacro" />
   <xacro:macro name="tomato" params="tomato_name radius parent_link *origin">
-    <xacro:property name = "rho" value="1000"/> <!-- [kg/m^3]-->
+    <xacro:property name = "rho" value="1"/> <!-- [kg/m^3]-->
     <xacro:property name = "V" value="${4/3*pi*radius**3}"/> <!-- [m^3]-->
     <xacro:property name = "mass" value="${rho * V}"/> <!-- [kg]-->

Commit message: Fixed some angle defintion, everything now works in both debugging and non-debugging mode for the object detection.

File: flex_gazebo/urdf/truss/3d/peduncle.xacro (robot description, xacro)
@@ -14,5 +14,5 @@
       <collision>
         <!-- origin is in the center of the cylinder-->
-        <origin xyz="0 0 0" rpy="${pi/2} 0 0"/>
+        <origin xyz="0 0 0" rpy="0 ${pi/2} 0"/>
         <geometry>
           <cylinder radius="${peduncle_radius}" length="${peduncle_length}"/>
@@ -20,5 +20,5 @@
       </collision>
       <visual>
-        <origin xyz="0 0 0" rpy="${pi/2} 0 0"/>
+        <origin xyz="0 0 0" rpy="0 ${pi/2} 0"/>
         <geometry>
           <cylinder radius="${peduncle_radius}" length="${peduncle_length}"/>

File: flex_gazebo/urdf/truss/3d/truss.xacro (robot description, xacro)
@@ -8,10 +8,12 @@
     <xacro:property name="peduncle_length" value="0.1" />
     <xacro:property name="peduncle_radius" value="0.01" />
-    <xacro:peduncle peduncle_length="${peduncle_length}" peduncle_radius="${peduncle_radius}" parent_link="world"/>
+    <xacro:peduncle peduncle_length="${peduncle_length}"
+      peduncle_radius="${peduncle_radius}"
+      parent_link="world"/>
     <xacro:tomato tomato_name="1" radius="${tomato_radius}" parent_link="peduncle">
-          <origin xyz="0 ${peduncle_length/2 + tomato_radius} 0" rpy="0 0 0" />
+          <origin xyz="${peduncle_length/2 + tomato_radius} 0 0" rpy="0 0 0" />
     </xacro:tomato>
     <xacro:tomato tomato_name="2" radius="${tomato_radius}" parent_link="peduncle">
-          <origin xyz="0 ${-peduncle_length/2 - tomato_radius} 0" rpy="0 0 0" />
+          <origin xyz="${-peduncle_length/2 - tomato_radius} 0 0" rpy="0 0 0" />
     </xacro:tomato>
   </xacro:macro>
