Commit message: Tracking aruco marker

File: flex_gazebo/urdf/marker/marker.xacro (robot description, xacro)
@@ -2,7 +2,6 @@
 <robot xmlns:xacro="http://www.ros.org/wiki/xacro">
 <xacro:include filename="$(find flex_gazebo)/urdf/marker/marker.gazebo.xacro" />
-  <xacro:macro name="marker" params="parent_link size *origin">
-    <xacro:property name = "ID" value="26"/>
-    <xacro:property name = "xyz" value="-0.01 0 0.035"/>
+  <xacro:macro name="marker" params="parent_link size ID *origin">
+    <xacro:property name = "xyz" value="-0.02 0 0.036"/>
     <joint name="marker__${ID}_joint" type="fixed">
       <xacro:insert_block name="origin" />

File: flex_gazebo/urdf/robot.urdf.xacro (robot description, xacro)
@@ -64,5 +64,5 @@
     </xacro:px150>
   </xacro:if>
-  <xacro:marker parent_link="px150/ee_arm_link" size="0.02">
+  <xacro:marker parent_link="px150/ee_arm_link" size="0.04" ID ="26" >
     <origin xyz="$(arg marker_origin_xyz)" rpy="$(arg marker_origin_rpy)" />
   </xacro:marker>

Commit message: Fixed calibration, was using incorect marker size

File: flex_gazebo/urdf/marker/marker.xacro (robot description, xacro)
@@ -4,4 +4,8 @@
   <xacro:macro name="marker" params="parent_link size ID *origin">
     <xacro:property name = "xyz" value="0 0 0"/>
+    <xacro:property name = "rpy" value="0 0 0"/>
+    <xacro:property name = "t" value="0.001"/>
+    <xacro:property name = "c" value="${1 + 2/15}"/>
+    <xacro:property name = "dim" value="${c * size} ${c * size} ${t}"/>
     <joint name="marker__${ID}_joint" type="fixed">
       <xacro:insert_block name="origin" />
@@ -11,19 +15,19 @@
     <link name="marker_${ID}">
       <inertial>
-        <origin xyz="${xyz}" rpy="0 0 0"/>
+        <origin xyz="${xyz}" rpy="${rpy}"/>
         <mass value="0.001"/>
         <inertia ixx="0"  ixy="0"  ixz="0" iyy="0" iyz="0" izz="0" />
       </inertial>
       <visual>
-        <origin xyz="${xyz}" rpy="0 0 0"/>
+        <origin xyz="${xyz}" rpy="${rpy}"/>
         <geometry>
-          <box size="${size} ${size} 0.001"/>
+          <box size="${dim}"/>
         </geometry>
         <materia name="Marker"/> <!-- Aruco/marker26_8cm -->
       </visual>
       <collision>
-        <origin xyz="${xyz}" rpy="0 0 0"/>
+        <origin xyz="${xyz}" rpy="${rpy}"/>
         <geometry>
-          <box size="${size} ${size} 0.001"/>
+          <box size="${dim}"/>
         </geometry>
       </collision>
