Commit message: Working on Communication class, most functionalities work again, Not fully implemented yet!

File: flex_gazebo_interbotix/urdf/experiments.urdf.xacro (robot description, xacro)
@@ -6,5 +6,6 @@
   <parent link="world"/>
   <child link="$(arg robot_name)/base_link"/>
-  <origin rpy="0 ${radians(3)} 0" xyz="0 0 0.005"/>
+  <!-- <origin rpy="0 ${radians(3)} 0" xyz="0 0 0.005"/> -->
+  <origin rpy="0 0 0" xyz="0 0 0"/>
 </joint>
 </robot>

Commit message: We may define pose_transform with respect to a different frame than the planning frame

File: flex_gazebo_interbotix/urdf/experiments.urdf.xacro (robot description, xacro)
@@ -6,6 +6,6 @@
   <parent link="world"/>
   <child link="$(arg robot_name)/base_link"/>
-  <!-- <origin rpy="0 ${radians(3)} 0" xyz="0 0 0.005"/> -->
-  <origin rpy="0 0 0" xyz="0 0 0"/>
+  <origin rpy="0 ${radians(3)} 0" xyz="0 0 0.005"/>
+  <!-- <origin rpy="0 0 0" xyz="0 0 0"/> -->
 </joint>
 </robot>

Commit message: Added pid control

File: flex_gazebo_interbotix/urdf/experiments.urdf.xacro (robot description, xacro)
@@ -6,6 +6,6 @@
   <parent link="world"/>
   <child link="$(arg robot_name)/base_link"/>
-  <origin rpy="0 ${radians(3)} 0" xyz="0 0 0.005"/>
-  <!-- <origin rpy="0 0 0" xyz="0 0 0"/> -->
+  <!-- <origin rpy="0 ${radians(3)} 0" xyz="0 0 0.005"/> -->
+  <origin rpy="0 0 0" xyz="0 0 0"/>
 </joint>
 </robot>
