Commit message: Can now modify camera resolution of simulation

File: flex_gazebo/urdf/camera/camera.gazebo.xacro (robot description, xacro)
@@ -1,5 +1,5 @@
 <?xml version="1.0"?>
 <robot xmlns:xacro="http://www.ros.org/wiki/xacro">
-  <xacro:macro name="my_camera" params="name">
+  <xacro:macro name="my_camera" params="name depth_width depth_height color_width color_height">
     <!-- Link1 -->
     <gazebo reference="${name}_color_frame"> <!--  -->
@@ -9,6 +9,6 @@
           <horizontal_fov>1.047</horizontal_fov>
           <image>
-            <width>1920</width>
-            <height>1080</height>
+            <width>${color_width}</width>
+            <height>${color_height}</height>
             <format>RGB_INT8</format>
           </image>
@@ -47,5 +47,5 @@
     </gazebo>
     <!-- Depth frame-->
-    <!-- TODO: reference frame is incorrect -->
+    <!-- TODO: if aligned_depth_to_color == true: camera_color_frame, else: camera_depth_frame  -->
     <gazebo reference="${name}_color_frame">
       <sensor name="depth" type="depth">
@@ -54,6 +54,6 @@
           <horizontal_fov>1.047</horizontal_fov>
           <image>
-            <width>1920</width>
-            <height>1080</height>
+            <width>${depth_width}</width>
+            <height>${depth_height}</height>
           </image>
           <clip>

File: flex_gazebo_interbotix/urdf/robot.urdf.xacro (robot description, xacro)
@@ -7,15 +7,19 @@
   <xacro:include filename="$(find flex_gazebo)/urdf/camera/camera.gazebo.xacro" />
   <!-- px150 params-->
-  <xacro:arg name="hardware_interface" default="PositionJointInterface"/>
-  <xacro:arg name="robot_name" default="px150"/>
-  <xacro:arg name="robot_model" default="px150"/>
-  <xacro:arg name="interbotix_origin_xyz" default="-0.2 0.45 0.23"/>
-  <xacro:arg name="interbotix_origin_rpy" default="0.0 0.0 0.0"/>
+  <xacro:arg name="hardware_interface"      default="PositionJointInterface"/>
+  <xacro:arg name="robot_name"              default="px150"/>
+  <xacro:arg name="robot_model"             default="px150"/>
+  <xacro:arg name="interbotix_origin_xyz"   default="-0.2 0.45 0.23"/>
+  <xacro:arg name="interbotix_origin_rpy"   default="0.0 0.0 0.0"/>
   <!-- camera params-->
-  <xacro:arg name="camera_name" default="rs_d435"/>
-  <xacro:arg name="camera_sim" default="true"/>
-  <xacro:arg name="use_nominal_extrinsics" default="$(arg camera_sim)"/>
-  <xacro:arg name="camera_origin_xyz" default="0.1 0.45 0.9"/>
-  <xacro:arg name="camera_origin_rpy" default="3.1415 1.57 -1.57"/>
+  <xacro:arg name="camera_name"             default="rs_d435"/>
+  <xacro:arg name="camera_sim"              default="true"/>
+  <xacro:arg name="use_nominal_extrinsics"  default="$(arg camera_sim)"/>
+  <xacro:arg name="camera_origin_xyz"       default="0.1 0.45 0.9"/>
+  <xacro:arg name="camera_origin_rpy"       default="3.1415 1.57 -1.57"/>
+  <xacro:arg name="depth_width"             default="1280"/>
+  <xacro:arg name="depth_height"            default="720"/>
+  <xacro:arg name="color_width"             default="1280"/>
+  <xacro:arg name="color_height"            default="720"/>
   <!-- marker -->
   <xacro:arg name="marker_origin_xyz" default="-0.02 0 0.036"/>
@@ -36,9 +40,21 @@
   </xacro:marker>
   <!-- camera -->
-  <xacro:sensor_d435 parent="world" name="$(arg camera_name)" use_nominal_extrinsics="$(arg use_nominal_extrinsics)">
-    <origin xyz="$(arg camera_origin_xyz)" rpy="$(arg camera_origin_rpy)" />
+  <xacro:sensor_d435
+    parent="world"
+    name="$(arg camera_name)"
+    use_nominal_extrinsics="$(arg use_nominal_extrinsics)">
+    <origin
+      xyz="$(arg camera_origin_xyz)"
+      rpy="$(arg camera_origin_rpy)"
+    />
   </xacro:sensor_d435>
   <xacro:if value="$(arg camera_sim)">
-    <xacro:my_camera name="$(arg camera_name)"/>
+    <xacro:my_camera
+      name="$(arg camera_name)"
+      depth_width="$(arg depth_width)"
+      depth_height="$(arg depth_height)"
+      color_width="$(arg color_width)"
+      color_height="$(arg color_height)"
+    />
   </xacro:if>
 </robot>
